File: simp.kicad_sch (KiCad schematic)
At the start: 54 parts, among them J1 AVR-ISP-6, J2 I2C, J3 USB_C_Receptacle_USB2.0, SW1 MX_SW_solder, SW10 MX_SW_solder, SW11 MX_SW_solder, SW12 MX_SW_solder, SW13 MX_SW_solder, SW14 MX_SW_solder, SW15 MX_SW_solder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

Commit message: version: bump version to 1.0.0
Other:
- company:  leonbcode -> leonbcode
